File: KSGER Controller/KSGER Controller/KSGER Controller.kicad_sch (KiCad schematic)
At the start: 14 parts

Commit message: Done for the night
Parts:
- added C3: 100 16V, symbol Device:C_Polarized
- added C4, C7: 0.1, symbol Device:C
- added D2: 1N4148WS, Diode_SMD:D_SOD-323, symbol Diode:1N4148WS
- added J?: 24 VDC, symbol Connector_Generic:Conn_01x02
- added J?: IRON_IN, symbol Connector_Generic:Conn_01x05
- added Q2: S8050, Package_TO_SOT_THT:TO-92_Inline, symbol Transistor_BJT:S8050
- added R11: 4.7K, symbol Device:R_Small
- added R13: 4.7k, symbol Device:R_Small
- added R14, R2: 6R8, symbol Device:R_Small
- added R8: 10K, symbol Device:R_Small
- added R9: 1K, symbol Device:R_Small
- added U2: AMS1117-3.3, Package_TO_SOT_SMD:SOT-223-3_TabPin2, symbol Regulator_Linear:AMS1117-3.3
- added U4: 24LC08, symbol Memory_EEPROM:24LC08
- added U6: L78L08_SOT89, Package_TO_SOT_SMD:SOT-89-3, symbol Regulator_Linear:L78L08_SOT89
- added U7: SSD1106, KSGER Controller Parts Library:SSD1106, symbol KSGER Controller Parts:SSD1106
- BT1: value (none) -> CR2032
- BZ1: value (none) -> Buzzer
- C1, C10, C11: value (none) -> 0.1
- J1: value (none) -> SWD
- J4: value (none) -> BATT
- J6: value (none) -> Conn_01x02_Female
- R10: value (none) -> 4.7K; symbol Device:R -> Device:R_Small
- SW1: value (none) -> ENCODER
- U1: value (none) -> STM32F103C8Tx; footprint (none) -> Package_QFP:LQFP-48_7x7mm_P0.5mm
- Y1: value (none) -> 32.768MHz
Connections:
- net +3V3: now also C3.1, C4.1, R11.1, R13.1, R2.1, U2.2 (VO), U4.8 (VCC)
- net EE_SCL: now also U4.6 (SCL)
- net EE_SDA: now also R11.2, R13.2, U4.5 (SDA)
- net GND: now also C3.2, C4.2, C7.2, J?.1 (Pin_1), R9.1, U2.1 (GND), U4.1 (A0), U4.2 (A1), U4.3 (A2), U4.4 (GND), U6.2 (GND), U7.2 (GND)
- net OLED_SCL: now also U7.3 (SCL)
- net OLED_SDA: now also U7.4 (SDA)
- net VIN_MON: now also C7.1, R8.1, R9.2
- new net: D2.2 (A), J?.2 (Pin_2), R8.2
- new net: U2.3 (VI), U6.1 (OUT)
- new net: R14.2, U6.3 (IN)
- new net: R2.2, U7.1 (VCC)
- new net: D2.1 (K), R14.1
- no-connect marks 18 -> 19
Other:
- moved on the sheet: BT1, BZ1, C1, C10, C11, J1, J4, R10, SW1, U1, Y1

Commit message: Finished schematic
Parts:
- removed BT1: CR2032, symbol Device:Battery_Cell
- removed J6: Conn_01x02_Female, symbol Connector:Conn_01x02_Female
- added C12: (no value), symbol Device:C
- added D1: (no value), symbol Device:LED
- added D3: (no value), symbol Diode:1N5819
- added Q1: (no value), symbol KSGER Controller Parts:IRF7416
- added R1, R12, R15, R16, R17, R18, R3, R4, R5, R6, R7: (no value), symbol Device:R
- added U3: (no value), symbol KSGER Controller Parts:SGM8551
- BZ1: value Buzzer -> (none)
- C1, C10, C11, C4, C7: value 0.1 -> (none); JCLPCB Part # (none) -> C49678
- C3: value 100 16V -> (none); JCLPCB Part # (none) -> C129274
- D2: value 1N4148WS -> (none); footprint Diode_SMD:D_SOD-323 -> (none); JCLPCB Part # (none) -> C2128
- J1: renamed from J?; value 24 VDC -> (none)
- J2: renamed from J?; value IRON_IN -> (none)
- J4: value BATT -> (none)
- J5: renamed from J1; value SWD -> (none)
- Q2: value S8050 -> (none); footprint Package_TO_SOT_THT:TO-92_Inline -> (none); JCLPCB Part # (none) -> C2146
- R10, R11: value 4.7K -> (none); symbol Device:R_Small -> Device:R; JCLPCB Part # (none) -> C23162
- R13: value 4.7k -> (none); symbol Device:R_Small -> Device:R; JCLPCB Part # (none) -> C23162
- R14, R2: value 6R8 -> (none); symbol Device:R_Small -> Device:R; JCLPCB Part # (none) -> C23212
- R8: value 10K -> (none); symbol Device:R_Small -> Device:R; JCLPCB Part # (none) -> C25197
- R9: value 1K -> (none); symbol Device:R_Small -> Device:R; JCLPCB Part # (none) -> C21190
- SW1: value ENCODER -> (none); JCLPCB Part # (none) -> C278348
- U1: value STM32F103C8Tx -> (none); footprint Package_QFP:LQFP-48_7x7mm_P0.5mm -> (none); JCLPCB Part # (none) -> C8734
- U2: value AMS1117-3.3 -> (none); footprint Package_TO_SOT_SMD:SOT-223-3_TabPin2 -> (none); JCLPCB Part # (none) -> C6186
- U4: value 24LC08 -> (none); JCLPCB Part # (none) -> C5455
- U6: value L78L08_SOT89 -> (none); footprint Package_TO_SOT_SMD:SOT-89-3 -> (none); JCLPCB Part # (none) -> C472525
- U7: value SSD1106 -> (none); footprint KSGER Controller Parts Library:SSD1106 -> (none)
- Y1: value 32.768MHz -> (none); JCLPCB Part # (none) -> C369191
Connections:
- net +3V3: now also R15.1, R17.1, R18.1, U3.5 (V+)
- net GND: now also J2.3 (Pin_3), J2.4 (Pin_4), Q2.1 (E), D1.1 (K), D3.2 (A), R6.2, R7.2, U3.2 (V-)
- net HEATER_ON: now also Q2.2 (B), R6.1
- net NTC: now also R12.2
- net SHAKE: now also R16.2
- net TIP_TEMP: now also R5.1, U3.1
- net at Q2.3 (C): now also R4.2
- net at J2.1 (Pin_1): now also R16.1, R17.2
- net at J2.2 (Pin_2): now also R12.1, R18.2
- net at J2.5 (Pin_5): now also C12.2, D3.1 (K), Q1.5, Q1.6, Q1.7, Q1.8, R1.2, R15.2
- net BUZZER: no longer names the net of BZ1.2 (+), U1.13 (PA3), U1.14 (PA4), U1.15 (PA5)
- new net: R5.2, R7.1, U3.4 (-)
- new net: Q1.4, R3.2, R4.1
- new net: D1.2 (A), R1.1, U3.3 (+)
- new net +24V: C12.1, Q1.1, Q1.2, Q1.3, R3.1
Other:
- note added: "+"
- note added: "CR2032"
- note added: "E"
- note added: "G"
- note added: "IRON INTERFACE"
- note added: "MCU"
- note added: "MEMORY"
- note added: "N"
- note added: "NOTE: C12 AND D3 ARE MODIFICATIONS OF THE ORIGINAL KSGER DESIGN ADDED BY MINSTORM88 THE FOLLOWING REFERENCES ARE DIFFERENT ON THIS DESIGN FROM MINDSTORM88'S DESIGN. MINDSTORM88'S REFERENCE IS ON THE LEFT: R12A - R12 R12B - R16 R12C - R17 R1B - R15 RX - R18"
- note added: "POWER SUPPLY"
- note added: "PRGM"
- note added: "S"
- note added: "USER INTERFACE AND DISPLAY"
- title: (none) -> KSGER T12 Soldering Iron Heating Controller
- moved on the sheet: BZ1, C1, C10, C11, C3, C4, C7, D2, J1, J2, J4, J5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

Commit message: more playing around
Parts:
- renumbered R10 to R19, R10 to R20
Other:
- note added: "NOTES: C12 AND D3 ARE MODIFICATIONS OF THE ORIGINAL KSGER DESIGN ADDED BY MINSTORM88 THE FOLLOWING REFERENCES ARE DIFFERENT ON THIS DESIGN FROM MINDSTORM88'S DESIGN. MINDSTORM88'S REFERENCE IS ON THE LEFT: R12A - R12 R12B - R16 R12C - R17 R1B - R15 RX - R18 R10 - THERE ARE 3 RESISTORS MARKED AS R10 ON THE ORIGINAL BOARD. TO STOP KICAD FROM THROWING AN ANNOTATION ERROR, I HAVE RENAMED TWO OF THEM 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"
- note removed: "NOTE: C12 AND D3 ARE MODIFICATIONS OF THE ORIGINAL KSGER DESIGN ADDED BY MINSTORM88 THE FOLLOWING REFERENCES ARE DIFFERENT ON THIS DESIGN FROM MINDSTORM88'S DESIGN. MINDSTORM88'S REFERENCE IS ON THE LEFT: R12A - R12 R12B - R16 R12C - R17 R1B - R15 RX - R18"
Changed lines of the file:
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@@
     (effects (font (size 1.27 1.27)) (justify left bottom))
   )
-  (text "NOTE:\nC12 AND D3 ARE MODIFICATIONS\nOF THE ORIGINAL KSGER DESIGN\nADDED BY MINSTORM88\n\nTHE FOLLOWING REFERENCES ARE DIFFERENT\nON THIS DESIGN FROM MINDSTORM88'S DESIGN.\nMINDSTORM88'S REFERENCE IS ON THE LEFT:\n\nR12A - R12\nR12B - R16\nR12C - R17\nR1B  - R15\nRX   - R18"
-    (at 247.65 280.67 0)
+  (text "NOTES:\n\nC12 AND D3 ARE MODIFICATIONS\nOF THE ORIGINAL KSGER DESIGN\nADDED BY MINSTORM88\n\nTHE FOLLOWING REFERENCES ARE DIFFERENT\nON THIS DESIGN FROM MINDSTORM88'S DESIGN.\nMINDSTORM88'S REFERENCE IS ON THE LEFT:\n\nR12A - R12\nR12B - R16\nR12C - R17\nR1B  - R15\nRX   - R18\n\nR10 - THERE ARE 3 RESISTORS MARKED AS R10 ON\nTHE ORIGINAL BOARD.  TO STOP KICAD FROM THROWING\nAN ANNOTATION ERROR, I HAVE RENAMED TWO OF \nTHEM TO R19 AND R20."
+    (at 233.68 279.4 0)
     (effects (font (size 1.27 1.27)) (justify left bottom))
   )
@@
   (symbol (lib_id "Device:R") (at 109.22 227.33 0) (mirror y) (unit 1)
     (in_bom yes) (on_board yes)
-    (property "Reference" "R10" (id 0) (at 106.68 229.87 90)
+    (property "Reference" "R20" (id 0) (at 106.68 229.87 90)
       (effects (font (size 1.27 1.27)) (justify left))
     )
@@
   (symbol (lib_id "Device:R") (at 104.14 227.33 0) (mirror y) (unit 1)
     (in_bom yes) (on_board yes)
-    (property "Reference" "R10" (id 0) (at 101.6 229.87 90)
+    (property "Reference" "R19" (id 0) (at 101.6 229.87 90)
       (effects (font (size 1.27 1.27)) (justify left))
     )
@@
       (reference "R9") (unit 1) (value "1K") (footprint "Resistor_SMD:R_0603_1608Metric")
     )
-    (path "/1c3992b6-8267-4680-adab-d2ce2dfdb302"
-      (reference "R10") (unit 1) (value "4.7K") (footprint "Resistor_SMD:R_0603_1608Metric")
-    )
-    (path "/27d91a52-75c3-47e1-bf8e-a246027d2e7b"
-      (reference "R10") (unit 1) (value "4.7K") (footprint "Resistor_SMD:R_0603_1608Metric")
-    )
     (path "/3eff7e40-9026-4e04-9f87-df1243540b0f"
       (reference "R10") (unit 1) (value "4.7K") (footprint "Resistor_SMD:R_0603_1608Metric")
@@
       (reference "R18") (unit 1) (value "4.7K") (footprint "Resistor_SMD:R_0603_1608Metric")
     )
+    (path "/27d91a52-75c3-47e1-bf8e-a246027d2e7b"
+      (reference "R19") (unit 1) (value "4.7K") (footprint "Resistor_SMD:R_0603_1608Metric")
+    )
+    (path "/1c3992b6-8267-4680-adab-d2ce2dfdb302"
+      (reference "R20") (unit 1) (value "4.7K") (footprint "Resistor_SMD:R_0603_1608Metric")
+    )
     (path "/f14c38dc-3541-4bf1-bafb-f86ba702358a"
       (reference "SW1") (unit 1) (value "ENCODER") (footprint "Rotary_Encoder:RotaryEncoder_Alps_EC11E-Switch_Vertical_H20mm")
@@
     )
     (path "/484b5dcd-a371-4568-b6e2-0bf747f30fdf"
-      (reference "U4") (unit 1) (value "24LC08") (footprint "Package_SO:SOIC-8-1EP_3.9x4.9mm_P1.27mm_EP2.62x3.51mm")
+      (reference "U4") (unit 1) (value "24LC08") (footprint "Package_SO:SOP-8_3.9x4.9mm_P1.27mm")
     )
     (path "/135f0285-24f7-4de4-affa-68f14431ec1e"

Commit message: Started working on PCB
Parts:
- added H1, H2, H3, H4: (no value), symbol Mechanical:MountingHole_Pad
Connections:
- net GND: now also H1.1, H2.1, H3.1, H4.1
Changed lines of the file:
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@@
   (junction (at 63.5 53.34) (diameter 0) (color 0 0 0 0)
   )
+  (junction (at 374.65 217.17) (diameter 0) (color 0 0 0 0)
+  )
   (junction (at 72.39 177.8) (diameter 0) (color 0 0 0 0)
   )
@@
   (junction (at 288.29 109.22) (diameter 0) (color 0 0 0 0)
   )
+  (junction (at 374.65 207.01) (diameter 0) (color 0 0 0 0)
+  )
   (junction (at 58.42 172.72) (diameter 0) (color 0 0 0 0)
   )
@@
   )
   (junction (at 331.47 139.7) (diameter 0) (color 0 0 0 0)
+  )
+  (junction (at 374.65 212.09) (diameter 0) (color 0 0 0 0)
   )
   (junction (at 100.33 248.92) (diameter 0) (color 0 0 0 0)
@@
     (stroke (width 0) (type default) (color 0 0 0 0))
   )
+  (wire (pts (xy 374.65 217.17) (xy 374.65 220.98))
+    (stroke (width 0) (type default) (color 0 0 0 0))
+  )
   (wire (pts (xy 100.33 259.08) (xy 100.33 260.35))
     (stroke (width 0) (type default) (color 0 0 0 0))
@@
     (stroke (width 0) (type default) (color 0 0 0 0))
   )
+  (wire (pts (xy 374.65 217.17) (xy 377.19 217.17))
+    (stroke (width 0) (type default) (color 0 0 0 0))
+  )
   (wire (pts (xy 149.86 177.8) (xy 138.43 177.8))
     (stroke (width 0) (type default) (color 0 0 0 0))
@@
     (stroke (width 0) (type default) (color 0 0 0 0))
   )
+  (wire (pts (xy 377.19 201.93) (xy 374.65 201.93))
+    (stroke (width 0) (type default) (color 0 0 0 0))
+  )
   (wire (pts (xy 86.36 41.91) (xy 92.71 41.91))
     (stroke (width 0) (type default) (color 0 0 0 0))
@@
     (stroke (width 0) (type default) (color 0 0 0 0))
   )
+  (wire (pts (xy 374.65 207.01) (xy 374.65 212.09))
+    (stroke (width 0) (type default) (color 0 0 0 0))
+  )
   (wire (pts (xy 189.23 179.07) (xy 187.96 179.07))
     (stroke (width 0) (type default) (color 0 0 0 0))
@@
     (stroke (width 0) (type default) (color 0 0 0 0))
   )
+  (wire (pts (xy 374.65 201.93) (xy 374.65 207.01))
+    (stroke (width 0) (type default) (color 0 0 0 0))
+  )
   (wire (pts (xy 104.14 218.44) (xy 104.14 220.98))
     (stroke (width 0) (type default) (color 0 0 0 0))
@@
     (stroke (width 0) (type default) (color 0 0 0 0))
   )
+  (wire (pts (xy 374.65 212.09) (xy 374.65 217.17))
+    (stroke (width 0) (type default) (color 0 0 0 0))
+  )
+  (wire (pts (xy 374.65 212.09) (xy 377.19 212.09))
+    (stroke (width 0) (type default) (color 0 0 0 0))
+  )
   (wire (pts (xy 46.99 67.31) (xy 46.99 54.61))
     (stroke (width 0) (type default) (color 0 0 0 0))
@@
   )
   (wire (pts (xy 109.22 231.14) (xy 109.22 240.03))
+    (stroke (width 0) (type default) (color 0 0 0 0))
+  )
+  (wire (pts (xy 374.65 207.01) (xy 377.19 207.01))
     (stroke (width 0) (type default) (color 0 0 0 0))
   )
@@
     (pin "2")
   )
+  (symbol (lib_id "Mechanical:MountingHole_Pad") (at 379.73 207.01 270) (unit 1)
+    (in_bom yes) (on_board yes) (fields_autoplaced)
+    (property "Reference" "H2" (id 0) (at 383.54 205.7399 90)
+      (effects (font (size 1.27 1.27)) (justify left))
+    )
+    (property "Value" "" (id 1) (at 383.54 208.2799 90)
+      (effects (font (size 1.27 1.27)) (justify left))
+    )
+    (property "Footprint" "" (id 2) (at 379.73 207.01 0)
+      (effects (font (size 1.27 1.27)) hide)
+    )
+    (property "Datasheet" "~" (id 3) (at 379.73 207.01 0)
+      (effects (font (size 1.27 1.27)) hide)
+    )
+    (pin "1")
+  )
   (symbol (lib_id "power:GND") (at 309.88 177.8 0) (unit 1)
     (in_bom yes) (on_board yes) (fields_autoplaced)
@@
     (pin "1")
   )
+  (symbol (lib_id "Mechanical:MountingHole_Pad") (at 379.73 212.09 270) (unit 1)
+    (in_bom yes) (on_board yes) (fields_autoplaced)
+    (property "Reference" "H3" (id 0) (at 383.54 210.8199 90)
+      (effects (font (size 1.27 1.27)) (justify left))
+    )
+    (property "Value" "" (id 1) (at 383.54 213.3599 90)
+      (effects (font (size 1.27 1.27)) (justify left))
+    )
+    (property "Footprint" "" (id 2) (at 379.73 212.09 0)
+      (effects (font (size 1.27 1.27)) hide)
+    )
+    (property "Datasheet" "~" (id 3) (at 379.73 212.09 0)
+      (effects (font (size 1.27 1.27)) hide)
+    )
+    (pin "1")
+  )
   (symbol (lib_id "Device:R") (at 153.67 177.8 270) (mirror x) (unit 1)
     (in_bom yes) (on_board yes)
@@
     (pin "3")
     (pin "4")
+  )
+  (symbol (lib_id "power:GND") (at 374.65 220.98 0) (unit 1)
+    (in_bom yes) (on_board yes) (fields_autoplaced)
+    (property "Reference" "#PWR01" (id 0) (at 374.65 227.33 0)
+      (effects (font (size 1.27 1.27)) hide)
+    )
+    (property "Value" "GND" (id 1) (at 374.65 226.06 0))
+    (property "Footprint" "" (id 2) (at 374.65 220.98 0)
+      (effects (font (size 1.27 1.27)) hide)
+    )
+    (property "Datasheet" "" (id 3) (at 374.65 220.98 0)
+      (effects (font (size 1.27 1.27)) hide)
+    )
+    (pin "1")
   )
   (symbol (lib_id "Device:R") (at 222.25 166.37 0) (mirror y) (unit 1)
@@
     (pin "1")
   )
+  (symbol (lib_id "Mechanical:MountingHole_Pad") (at 379.73 201.93 270) (unit 1)
+    (in_bom yes) (on_board yes) (fields_autoplaced)
+    (property "Reference" "H1" (id 0) (at 383.54 200.6599 90)
+      (effects (font (size 1.27 1.27)) (justify left))
+    )
+    (property "Value" "" (id 1) (at 383.54 203.1999 90)
+      (effects (font (size 1.27 1.27)) (justify left))
+    )
+    (property "Footprint" "" (id 2) (at 379.73 201.93 0)
+      (effects (font (size 1.27 1.27)) hide)
+    )
+    (property "Datasheet" "~" (id 3) (at 379.73 201.93 0)
+      (effects (font (size 1.27 1.27)) hide)
+    )
+    (pin "1")
+  )
   (symbol (lib_id "power:GND") (at 63.5 146.05 0) (unit 1)
     (in_bom yes) (on_board yes) (fields_autoplaced)
@@
     (pin "1")
     (pin "2")
+  )
+  (symbol (lib_id "Mechanical:MountingHole_Pad") (at 379.73 217.17 270) (unit 1)
+    (in_bom yes) (on_board yes) (fields_autoplaced)
+    (property "Reference" "H4" (id 0) (at 383.54 215.8999 90)
+      (effects (font (size 1.27 1.27)) (justify left))
+    )
+    (property "Value" "" (id 1) (at 383.54 218.4399 90)
+      (effects (font (size 1.27 1.27)) (justify left))
+    )
+    (property "Footprint" "" (id 2) (at 379.73 217.17 0)
+      (effects (font (size 1.27 1.27)) hide)
+    )
+    (property "Datasheet" "~" (id 3) (at 379.73 217.17 0)
+      (effects (font (size 1.27 1.27)) hide)
+    )
+    (pin "1")
   )
   (symbol (lib_id "Device:RotaryEncoder_Switch") (at 87.63 242.57 0) (mirror y) (unit 1)
@@
   )
   (symbol_instances
+    (path "/bd86cfc3-bdb1-4b21-95d4-5729326f1cc3"
+      (reference "#PWR01") (unit 1) (value "GND") (footprint "")
+    )
     (path "/b0ecd235-6b6f-47d7-b3af-f913e4e61f0e"
       (reference "#PWR0101") (unit 1) (value "GND") (footprint "")
@@
       (reference "D3") (unit 1) (value "1N5819") (footprint "Diode_SMD:D_SOD-323")
     )
+    (path "/e2581823-bdc7-40ad-9270-e8ded3a51138"
+      (reference "H1") (unit 1) (value "MountingHole_Pad") (footprint "MountingHole:MountingHole_3.2mm_M3_Pad_Via")
+    )
+    (path "/406ba619-a733-4fe8-8d85-324ff1a9b2a5"
+      (reference "H2") (unit 1) (value "MountingHole_Pad") (footprint "MountingHole:MountingHole_3.2mm_M3_Pad_Via")
+    )
+    (path "/b93c5547-d762-41bf-bac4-e1851c1a959c"
+      (reference "H3") (unit 1) (value "MountingHole_Pad") (footprint "MountingHole:MountingHole_3.2mm_M3_Pad_Via")
+    )
+    (path "/ee3af1dd-9b9e-4e2f-8f7d-58e38c690410"
+      (reference "H4") (unit 1) (value "MountingHole_Pad") (footprint "MountingHole:MountingHole_3.2mm_M3_Pad_Via")
+    )
     (path "/28576217-cca0-45a7-96c3-aa04baa17a8b"
