File: KSGER Controller.kicad_sch (KiCad schematic)
At the start: 51 parts

Commit message: Updated PDF
Parts:
- BZ1: value (none) -> Buzzer; footprint (none) -> Connector_JST:JST_EH_B2B-EH-A_1x02_P2.50mm_Vertical
- C1, C12, C4, C5, C6, C7: value (none) -> 0.1; footprint (none) -> Capacitor_SMD:C_0805_2012Metric
- C10, C11: value (none) -> 0.001; footprint (none) -> Capacitor_SMD:C_0805_2012Metric
- C3: value (none) -> 100 16V; footprint (none) -> Capacitor_Tantalum_SMD:CP_EIA-7343-31_Kemet-D
- D1: value (none) -> GRN; footprint (none) -> LED_SMD:LED_0603_1608Metric
- D2: value (none) -> 1N4148WS; footprint (none) -> Diode_SMD:D_SOD-323
- D3: value (none) -> 1N5819; footprint (none) -> Diode_SMD:D_SOD-323
- H1, H2, H3, H4: value (none) -> MountingHole_Pad; footprint (none) -> MountingHole:MountingHole_3.2mm_M3_Pad_Via
- J1: value (none) -> 24 VDC; footprint (none) -> Connector_JST:JST_EH_B2B-EH-A_1x02_P2.50mm_Vertical
- J2: value (none) -> IRON_IN; footprint (none) -> Connector_JST:JST_EH_B5B-EH-A_1x05_P2.50mm_Vertical
- J4: value (none) -> BATT; footprint (none) -> Connector_JST:JST_EH_B2B-EH-A_1x02_P2.50mm_Vertical
- J5: value (none) -> SWD; footprint (none) -> Connector_JST:JST_EH_B4B-EH-A_1x04_P2.50mm_Vertical
- Q1: value (none) -> IRF7416; footprint (none) -> Package_SO:SO-8_3.9x4.9mm_P1.27mm
- Q2: value (none) -> S8050; footprint (none) -> Package_TO_SOT_SMD:SOT-23
- R1, R10, R11, R12, R13, R16, R17, R18, R19, R20, R3, R4, R6: value (none) -> 4.7K; footprint (none) -> Resistor_SMD:R_0603_1608Metric
- R14, R2: value (none) -> 6R8; footprint (none) -> Resistor_SMD:R_0603_1608Metric
- R15: value (none) -> 910K; footprint (none) -> Resistor_SMD:R_0805_2012Metric
- R5: value (none) -> 249K; footprint (none) -> Resistor_SMD:R_0805_2012Metric
- R7, R9: value (none) -> 1K; footprint (none) -> Resistor_SMD:R_0603_1608Metric
- R8: value (none) -> 10K; footprint (none) -> Resistor_SMD:R_0603_1608Metric
- SW1: value (none) -> ENCODER; footprint (none) -> Rotary_Encoder:RotaryEncoder_Alps_EC11E-Switch_Vertical_H20mm
- U1: value (none) -> STM32F103C8Tx; footprint (none) -> Package_QFP:LQFP-48_7x7mm_P0.5mm
- U2: value (none) -> AMS1117-3.3; footprint (none) -> Package_TO_SOT_SMD:SOT-223-3_TabPin2
- U3: value (none) -> SGM8551; footprint (none) -> Package_TO_SOT_SMD:SOT-23-5
- U4: value (none) -> 24LC08; footprint (none) -> Package_SO:SOP-8_3.9x4.9mm_P1.27mm
- U6: value (none) -> L78L08_SOT89; footprint (none) -> Package_TO_SOT_SMD:SOT-89-3
- U7: value (none) -> SSD1106; footprint (none) -> KSGER Controller Parts Library:SSD1106
- Y1: value (none) -> 32.768MHz; footprint (none) -> Crystal:Crystal_SMD_3215-2Pin_3.2x1.5mm
